File: hardware/apps.kicad_sch (KiCad schematic)
At the start: 22 parts, among them SW1 SW_Push, U1 STM32L4P5RET6, Y1 8Mhz

Commit message: Refactor
Parts:
- SW1: value SW_Push -> Reset
Connections:
- net 3V3_A renamed VDDA
- net 3V3_SYS renamed +3V3
- net BRAKE_PRESSURE1 renamed BRK_PRESS1
- net BRAKE_PRESSURE2 renamed BRK_PRESS2
- net SENSOR1 renamed APPS1
- net SENSOR2 renamed APPS2
Other:
- sheet Potentiometers' Amplifiers renamed APPS
- sheet APPS: file AnalogInputs.kicad_sch -> analog_inputs.kicad_sch
- sheet APPS ports: added OUT1, OUT2; removed 3V3_POT1, 3V3_POT2, SENSOR1, SENSOR2
- sheet Brake Pressure Left ports: added none; removed 3V3_SYS
- sheet Brake Pressure Right ports: added none; removed 3V3_SYS
- sheet CAN Transceiver: file CAN.kicad_sch -> can_transceiver.kicad_sch
- sheet CAN Transceiver ports: added CAN_H, CAN_L, CAN_RX, CAN_TX; removed 3V3_SYS, CAN-H, CAN-L, CAN-RX, CAN-TX
- sheet Connectors: file Connectros.kicad_sch -> connectors.kicad_sch
- sheet Power: file PowerModule.kicad_sch -> power_module.kicad_sch
- sheet Power ports: added none; removed 3V3_POT1, 3V3_POT2, 3V3_SYS
- sheet Safety Relay: file Safety.kicad_sch -> safety_relay.kicad_sch
- sheet Safety Relay ports: added IN, OUT; removed SAFETY1, SAFETY2
- moved on the sheet: C1, C2, C3, C4, C5, C6, C7, C8, D1, D2, D3, D4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

Commit message: Update component values
Parts:
- D1, D2, D3, D4: value LED -> Yellow
- Y1: value 8Mhz -> 8MHz
Changed lines of the file:
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@@
   (symbol (lib_id "Device:R") (at 97.79 180.34 90) (unit 1)
     (in_bom yes) (on_board yes) (dnp no)
-    (property "Reference" "R5" (at 100.33 182.88 90)
-      (effects (font (size 1.27 1.27)))
-    )
-    (property "Value" "300R" (at 95.25 182.88 90)
+    (property "Reference" "R5" (at 95.25 182.88 90)
+      (effects (font (size 1.27 1.27)))
+    )
+    (property "Value" "300R" (at 100.33 182.88 90)
       (effects (font (size 1.27 1.27)))
     )
@@
   (symbol (lib_id "Device:R") (at 97.79 172.72 270) (unit 1)
     (in_bom yes) (on_board yes) (dnp no)
-    (property "Reference" "R4" (at 100.33 175.26 90)
-      (effects (font (size 1.27 1.27)))
-    )
-    (property "Value" "300R" (at 95.25 175.26 90)
+    (property "Reference" "R4" (at 95.25 175.26 90)
+      (effects (font (size 1.27 1.27)))
+    )
+    (property "Value" "300R" (at 100.33 175.26 90)
       (effects (font (size 1.27 1.27)))
     )
@@
   (symbol (lib_id "Device:R") (at 97.79 165.1 270) (unit 1)
     (in_bom yes) (on_board yes) (dnp no)
-    (property "Reference" "R3" (at 100.33 167.64 90)
-      (effects (font (size 1.27 1.27)))
-    )
-    (property "Value" "300R" (at 95.25 167.64 90)
+    (property "Reference" "R3" (at 95.25 167.64 90)
+      (effects (font (size 1.27 1.27)))
+    )
+    (property "Value" "300R" (at 100.33 167.64 90)
       (effects (font (size 1.27 1.27)))
     )
@@
       (effects (font (size 1.27 1.27)))
     )
-    (property "Value" "LED" (at 110.49 182.88 0)
+    (property "Value" "Yellow" (at 113.03 182.88 0)
       (effects (font (size 1.27 1.27)))
     )
@@
       (effects (font (size 1.27 1.27)))
     )
-    (property "Value" "LED" (at 110.49 175.26 0)
+    (property "Value" "Yellow" (at 113.03 175.26 0)
       (effects (font (size 1.27 1.27)))
     )
@@
       (effects (font (size 1.27 1.27)))
     )
-    (property "Value" "LED" (at 110.49 167.64 0)
+    (property "Value" "Yellow" (at 113.03 167.64 0)
       (effects (font (size 1.27 1.27)))
     )
@@
       (effects (font (size 1.27 1.27)))
     )
-    (property "Value" "LED" (at 110.49 161.29 0)
+    (property "Value" "Yellow" (at 113.03 161.29 0)
       (effects (font (size 1.27 1.27)))
     )
@@
   (symbol (lib_id "Device:R") (at 97.79 158.75 90) (unit 1)
     (in_bom yes) (on_board yes) (dnp no)
-    (property "Reference" "R2" (at 100.33 161.29 90)
-      (effects (font (size 1.27 1.27)))
-    )
-    (property "Value" "300R" (at 95.25 161.29 90)
+    (property "Reference" "R2" (at 95.25 161.29 90)
+      (effects (font (size 1.27 1.27)))
+    )
+    (property "Value" "300R" (at 100.33 161.29 90)
       (effects (font (size 1.27 1.27)))
     )
@@
       (effects (font (size 1.27 1.27)) (justify right))
     )
-    (property "Value" "8Mhz" (at 48.26 161.29 0)
+    (property "Value" "8MHz" (at 48.26 161.29 0)
       (effects (font (size 1.27 1.27)) (justify right))
     )
