File: hardware/apps.kicad_pcb (KiCad board)
At the start: 2 copper layers, 100 x 75 mm, 130 parts, among them J1 Signals, J2 Diagnostics, J3 Power & CAN, K1 FINDER-30.22, Q1 BSS138, SW1 SW_Push, U1 STM32L4P5RET6, U10 LM1117-3.3, U11 MCP6002-xMC, U2 MCP6N11-005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

Commit message: Refactor
Parts:
- R15, R17: value TBD -> 6k
- R16, R18: value TBD -> 1k
- SW1: value SW_Push -> Reset
Connections:
- net /3V3_A renamed VDDA
- net /3V3_SYS renamed +3V3
- net /BRAKE_PRESSURE1 renamed /BRK_PRESS1
- net /BRAKE_PRESSURE2 renamed /BRK_PRESS2
- net /Power/VO_POT1 renamed Net-(U9-VO)
- net /Power/VO_POT2 renamed Net-(U10-VO)
- net /SENSOR1 renamed /APPS1
- net /SENSOR2 renamed /APPS2
- net CAN-H renamed CAN+
- net CAN-L renamed CAN-
- net SAFETY-IN renamed SAFETY_IN
- net SAFETY-OUT renamed SAFETY_OUT

Commit message: Update component values
Parts:
- D1, D2, D3, D4: value LED -> Yellow
- D8: value DIODE -> STPS340U
- Q1: value BSS138 -> BSN20
- R15, R17: value 6k -> 6k2
- Y1: value 8Mhz -> 8MHz
Changed lines of the file:
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@@
         (effects (font (size 1 1) (thickness 0.15)))
     )
-    (fp_text value "6k" (at 0 1.43 90) (layer "F.Fab")
+    (fp_text value "6k2" (at 0 1.43 90) (layer "F.Fab")
         (effects (font (size 1 1) (thickness 0.15)))
     )
@@
         (effects (font (size 1 1) (thickness 0.15)))
     )
-    (fp_text value "BSS138" (at 0 2.4 90) (layer "F.Fab")
+    (fp_text value "BSN20" (at 0 2.4 90) (layer "F.Fab")
         (effects (font (size 1 1) (thickness 0.15)))
     )
@@
         (effects (font (size 1 1) (thickness 0.15)))
     )
-    (fp_text value "LED" (at 0 1.43) (layer "F.Fab")
+    (fp_text value "Yellow" (at 0 1.43) (layer "F.Fab")
         (effects (font (size 1 1) (thickness 0.15)))
     )
@@
         (effects (font (size 1 1) (thickness 0.15)))
     )
-    (fp_text value "8Mhz" (at 0 2.45) (layer "F.Fab")
+    (fp_text value "8MHz" (at 0 2.45) (layer "F.Fab")
         (effects (font (size 1 1) (thickness 0.15)))
     )
@@
         (effects (font (size 1 1) (thickness 0.15)))
     )
-    (fp_text value "DIODE" (at 0 3.1) (layer "F.Fab")
+    (fp_text value "STPS340U" (at 0 3.1) (layer "F.Fab")
         (effects (font (size 1 1) (thickness 0.15)))
     )
@@
         (effects (font (size 1 1) (thickness 0.15)))
     )
-    (fp_text value "6k" (at 0 1.43 90) (layer "F.Fab")
+    (fp_text value "6k2" (at 0 1.43 90) (layer "F.Fab")
         (effects (font (size 1 1) (thickness 0.15)))
     )
@@
         (effects (font (size 1 1) (thickness 0.15)))
     )
-    (fp_text value "LED" (at 0 1.43) (layer "F.Fab")
+    (fp_text value "Yellow" (at 0 1.43) (layer "F.Fab")
         (effects (font (size 1 1) (thickness 0.15)))
     )
@@
         (effects (font (size 1 1) (thickness 0.15)))
     )
-    (fp_text value "LED" (at 0 1.43) (layer "F.Fab")
+    (fp_text value "Yellow" (at 0 1.43) (layer "F.Fab")
         (effects (font (size 1 1) (thickness 0.15)))
     )
@@
         (effects (font (size 1 1) (thickness 0.15)))
     )
-    (fp_text value "LED" (at 0 1.43) (layer "F.Fab")
+    (fp_text value "Yellow" (at 0 1.43) (layer "F.Fab")
         (effects (font (size 1 1) (thickness 0.15)))
     )

Commit message: Adjust component values
Parts:
- D5, D6: value D_TVS -> 24V
- F1, F2: value Fuse -> 500mA
- R15: value 6k2 -> 4k7
- R27, R40: value TBD -> 1k5
- R28, R41: value TBD -> 2k2
- R30: value 220R -> 330R
- R31: value 0R -> 220R
Connections:
- C10 pad 1: 3V3_POT2 -> (no net)
- C10 pad 2: GND -> (no net)
- C12 pad 1: 3V3_POT2 -> (no net)
- C12 pad 2: GND -> (no net)
Changed lines of the file:
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@@
         (effects (font (size 1 1) (thickness 0.15)))
     )
-    (fp_text value "0R" (at 0 1.43 90) (layer "F.Fab")
+    (fp_text value "220R" (at 0 1.43 90) (layer "F.Fab")
         (effects (font (size 1 1) (thickness 0.15)))
     )
@@
         (effects (font (size 1 1) (thickness 0.15)))
     )
-    (fp_text value "TBD" (at 0 1.43) (layer "F.Fab")
+    (fp_text value "1k5" (at 0 1.43) (layer "F.Fab")
         (effects (font (size 1 1) (thickness 0.15)))
     )
@@
     (fp_line (start 0.8 0.4) (end -0.8 0.4)
       (stroke (width 0.1) (type solid)) (layer "F.Fab"))
-    (pad "1" smd roundrect (at -0.8625 0 180) (size 1.075 0.95) (layers "F.Cu" "F.Paste" "F.Mask") (roundrect_rratio 0.25)
-      (net 12 "3V3_POT2") (pintype "passive"))
-    (pad "2" smd roundrect (at 0.8625 0 180) (size 1.075 0.95) (layers "F.Cu" "F.Paste" "F.Mask") (roundrect_rratio 0.25)
-      (net 1 "GND") (pintype "passive"))
+    (pad "1" smd roundrect (at -0.8625 0 180) (size 1.075 0.95) (layers "F.Cu" "F.Paste" "F.Mask") (roundrect_rratio 0.25))
+    (pad "2" smd roundrect (at 0.8625 0 180) (size 1.075 0.95) (layers "F.Cu" "F.Paste" "F.Mask") (roundrect_rratio 0.25))
     (model "${KICAD6_3DMODEL_DIR}/Capacitor_SMD.3dshapes/C_0603_1608Metric.wrl"
       (offset (xyz 0 0 0))
@@
         (effects (font (size 1 1) (thickness 0.15)))
     )
-    (fp_text value "TBD" (at 0 1.43) (layer "F.Fab")
+    (fp_text value "1k5" (at 0 1.43) (layer "F.Fab")
         (effects (font (size 1 1) (thickness 0.15)))
     )
@@
         (effects (font (size 1 1) (thickness 0.15)))
     )
-    (fp_text value "D_TVS" (at 0 1.43 90) (layer "F.Fab")
+    (fp_text value "24V" (at 0 1.43 90) (layer "F.Fab")
         (effects (font (size 1 1) (thickness 0.15)))
     )
@@
         (effects (font (size 1 1) (thickness 0.15)))
     )
-    (fp_text value "6k2" (at 0 1.43 90) (layer "F.Fab")
+    (fp_text value "4k7" (at 0 1.43 90) (layer "F.Fab")
         (effects (font (size 1 1) (thickness 0.15)))
     )
@@
         (effects (font (size 1 1) (thickness 0.15)))
     )
-    (fp_text value "TBD" (at 0 1.43) (layer "F.Fab")
+    (fp_text value "2k2" (at 0 1.43) (layer "F.Fab")
         (effects (font (size 1 1) (thickness 0.15)))
     )
@@
         (effects (font (size 1 1) (thickness 0.15)))
     )
-    (fp_text value "D_TVS" (at 0 1.43 -270) (layer "F.Fab")
+    (fp_text value "24V" (at 0 1.43 -270) (layer "F.Fab")
         (effects (font (size 1 1) (thickness 0.15)))
     )
@@
         (effects (font (size 1 1) (thickness 0.15)))
     )
-    (fp_text value "Fuse" (at 0 2.28 90) (layer "F.Fab")
+    (fp_text value "500mA" (at 0 2.28 90) (layer "F.Fab")
         (effects (font (size 1 1) (thickness 0.15)))
     )
@@
         (effects (font (size 1 1) (thickness 0.15)))
     )
-    (fp_text value "TBD" (at 0 1.43) (layer "F.Fab")
+    (fp_text value "2k2" (at 0 1.43) (layer "F.Fab")
         (effects (font (size 1 1) (thickness 0.15)))
     )
@@
     (fp_line (start 0.8 0.4) (end -0.8 0.4)
       (stroke (width 0.1) (type solid)) (layer "F.Fab"))
-    (pad "1" smd roundrect (at -0.8625 0) (size 1.075 0.95) (layers "F.Cu" "F.Paste" "F.Mask") (roundrect_rratio 0.25)
-      (net 12 "3V3_POT2") (pintype "passive"))
-    (pad "2" smd roundrect (at 0.8625 0) (size 1.075 0.95) (layers "F.Cu" "F.Paste" "F.Mask") (roundrect_rratio 0.25)
-      (net 1 "GND") (pintype "passive"))
+    (pad "1" smd roundrect (at -0.8625 0) (size 1.075 0.95) (layers "F.Cu" "F.Paste" "F.Mask") (roundrect_rratio 0.25))
+    (pad "2" smd roundrect (at 0.8625 0) (size 1.075 0.95) (layers "F.Cu" "F.Paste" "F.Mask") (roundrect_rratio 0.25))
     (model "${KICAD6_3DMODEL_DIR}/Capacitor_SMD.3dshapes/C_0603_1608Metric.wrl"
       (offset (xyz 0 0 0))
@@
         (effects (font (size 1 1) (thickness 0.15)))
     )
-    (fp_text value "220R" (at 0 1.43 90) (layer "F.Fab")
+    (fp_text value "330R" (at 0 1.43 90) (layer "F.Fab")
         (effects (font (size 1 1) (thickness 0.15)))
     )
@@
         (effects (font (size 1 1) (thickness 0.15)))
     )
-    (fp_text value "Fuse" (at 0 2.28 90) (layer "F.Fab")
+    (fp_text value "500mA" (at 0 2.28 90) (layer "F.Fab")
         (effects (font (size 1 1) (thickness 0.15)))
     )

Commit message: Use voltage followers for the brake pressure measurements
Parts:
- R23, R36: value 1k -> 0R
- R24, R37: value 10k -> 100R
- R25, R38: value 2k -> 100R
- R26, R39: value 2k -> 0R
- R27, R40: value 1k5 -> 3k3
- R28, R41: value 2k2 -> 0R
Connections:
- C10 pad 1: (no net) -> 3V3_POT2
- C10 pad 2: (no net) -> GND
- C12 pad 1: (no net) -> 3V3_POT2
- C12 pad 2: (no net) -> GND
Changed lines of the file:
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@@
     (property "Sheetfile" "brake_pressure.kicad_sch")
     (property "Sheetname" "Brake Pressure Right")
+    (property "dnp" "")
     (property "ki_description" "Resistor")
     (property "ki_keywords" "R res resistor")
@@
         (effects (font (size 1 1) (thickness 0.15)))
     )
-    (fp_text value "1k5" (at 0 1.43) (layer "F.Fab")
+    (fp_text value "3k3" (at 0 1.43) (layer "F.Fab")
         (effects (font (size 1 1) (thickness 0.15)))
     )
@@
     (fp_line (start 0.8 0.4) (end -0.8 0.4)
       (stroke (width 0.1) (type solid)) (layer "F.Fab"))
-    (pad "1" smd roundrect (at -0.8625 0 180) (size 1.075 0.95) (layers "F.Cu" "F.Paste" "F.Mask") (roundrect_rratio 0.25))
-    (pad "2" smd roundrect (at 0.8625 0 180) (size 1.075 0.95) (layers "F.Cu" "F.Paste" "F.Mask") (roundrect_rratio 0.25))
+    (pad "1" smd roundrect (at -0.8625 0 180) (size 1.075 0.95) (layers "F.Cu" "F.Paste" "F.Mask") (roundrect_rratio 0.25)
+      (net 12 "3V3_POT2") (pintype "passive"))
+    (pad "2" smd roundrect (at 0.8625 0 180) (size 1.075 0.95) (layers "F.Cu" "F.Paste" "F.Mask") (roundrect_rratio 0.25)
+      (net 1 "GND") (pintype "passive"))
     (model "${KICAD6_3DMODEL_DIR}/Capacitor_SMD.3dshapes/C_0603_1608Metric.wrl"
       (offset (xyz 0 0 0))
@@
     (property "Sheetfile" "brake_pressure.kicad_sch")
     (property "Sheetname" "Brake Pressure Left")
+    (property "dnp" "")
     (property "ki_description" "Resistor")
     (property "ki_keywords" "R res resistor")
@@
         (effects (font (size 1 1) (thickness 0.15)))
     )
-    (fp_text value "1k5" (at 0 1.43) (layer "F.Fab")
+    (fp_text value "3k3" (at 0 1.43) (layer "F.Fab")
         (effects (font (size 1 1) (thickness 0.15)))
     )
@@
         (effects (font (size 1 1) (thickness 0.15)))
     )
-    (fp_text value "1k" (at 0 1.43) (layer "F.Fab")
+    (fp_text value "0R" (at 0 1.43) (layer "F.Fab")
         (effects (font (size 1 1) (thickness 0.15)))
     )
@@
     (property "Sheetfile" "brake_pressure.kicad_sch")
     (property "Sheetname" "Brake Pressure Left")
+    (property "dnp" "")
     (property "ki_description" "Resistor")
     (property "ki_keywords" "R res resistor")
@@
         (effects (font (size 1 1) (thickness 0.15)))
     )
-    (fp_text value "10k" (at 0 1.43 180) (layer "F.Fab")
+    (fp_text value "100R" (at 0 1.43 180) (layer "F.Fab")
         (effects (font (size 1 1) (thickness 0.15)))
     )
@@
     (property "Sheetfile" "brake_pressure.kicad_sch")
     (property "Sheetname" "Brake Pressure Right")
+    (property "dnp" "")
     (property "ki_description" "Resistor")
     (property "ki_keywords" "R res resistor")
@@
         (effects (font (size 1 1) (thickness 0.15)))
     )
-    (fp_text value "10k" (at 0 1.43 180) (layer "F.Fab")
+    (fp_text value "100R" (at 0 1.43 180) (layer "F.Fab")
         (effects (font (size 1 1) (thickness 0.15)))
     )
@@
         (effects (font (size 1 1) (thickness 0.15)))
     )
-    (fp_text value "2k2" (at 0 1.43) (layer "F.Fab")
+    (fp_text value "0R" (at 0 1.43) (layer "F.Fab")
         (effects (font (size 1 1) (thickness 0.15)))
     )
@@
     (property "Sheetfile" "brake_pressure.kicad_sch")
     (property "Sheetname" "Brake Pressure Left")
+    (property "dnp" "")
     (property "ki_description" "Resistor")
     (property "ki_keywords" "R res resistor")
@@
         (effects (font (size 1 1) (thickness 0.15)))
     )
-    (fp_text value "2k" (at 0 1.43 180) (layer "F.Fab")
+    (fp_text value "100R" (at 0 1.43 180) (layer "F.Fab")
         (effects (font (size 1 1) (thickness 0.15)))
     )
@@
         (effects (font (size 1 1) (thickness 0.15)))
     )
-    (fp_text value "1k" (at 0 1.43) (layer "F.Fab")
+    (fp_text value "0R" (at 0 1.43) (layer "F.Fab")
         (effects (font (size 1 1) (thickness 0.15)))
     )
@@
         (effects (font (size 1 1) (thickness 0.15)))
     )
-    (fp_text value "2k" (at 0 1.43) (layer "F.Fab")
+    (fp_text value "0R" (at 0 1.43) (layer "F.Fab")
         (effects (font (size 1 1) (thickness 0.15)))
     )
@@
     (property "Sheetfile" "brake_pressure.kicad_sch")
     (property "Sheetname" "Brake Pressure Right")
+    (property "dnp" "")
     (property "ki_description" "Resistor")
     (property "ki_keywords" "R res resistor")
@@
         (effects (font (size 1 1) (thickness 0.15)))
     )
-    (fp_text value "2k" (at 0 1.43 180) (layer "F.Fab")
+    (fp_text value "100R" (at 0 1.43 180) (layer "F.Fab")
         (effects (font (size 1 1) (thickness 0.15)))
     )
@@
         (effects (font (size 1 1) (thickness 0.15)))
     )
-    (fp_text value "2k2" (at 0 1.43) (layer "F.Fab")
+    (fp_text value "0R" (at 0 1.43) (layer "F.Fab")
         (effects (font (size 1 1) (thickness 0.15)))
     )
@@
     (fp_line (start 0.8 0.4) (end -0.8 0.4)
       (stroke (width 0.1) (type solid)) (layer "F.Fab"))
-    (pad "1" smd roundrect (at -0.8625 0) (size 1.075 0.95) (layers "F.Cu" "F.Paste" "F.Mask") (roundrect_rratio 0.25))
-    (pad "2" smd roundrect (at 0.8625 0) (size 1.075 0.95) (layers "F.Cu" "F.Paste" "F.Mask") (roundrect_rratio 0.25))
+    (pad "1" smd roundrect (at -0.8625 0) (size 1.075 0.95) (layers "F.Cu" "F.Paste" "F.Mask") (roundrect_rratio 0.25)
+      (net 12 "3V3_POT2") (pintype "passive"))
+    (pad "2" smd roundrect (at 0.8625 0) (size 1.075 0.95) (layers "F.Cu" "F.Paste" "F.Mask") (roundrect_rratio 0.25)
+      (net 1 "GND") (pintype "passive"))
     (model "${KICAD6_3DMODEL_DIR}/Capacitor_SMD.3dshapes/C_0603_1608Metric.wrl"
       (offset (xyz 0 0 0))
@@
         (effects (font (size 1 1) (thickness 0.15)))
     )
-    (fp_text value "2k" (at 0 1.43) (layer "F.Fab")
+    (fp_text value "0R" (at 0 1.43) (layer "F.Fab")
         (effects (font (size 1 1) (thickness 0.15)))
     )
